File: electrical/Tekk_Card/Tekk_Card.kicad_pcb (KiCad board)
At the start: 2 copper layers, 88.9 x 50.8 mm, 20 parts, among them U2 TLV76733DRVx, U3 RP2040, U5 W25Q64JVSSIQ

Commit message: Continue initial prototype
Parts:
- removed D13, D14, D15, D16, D17, D18: WS2812B, LED_SMD:LED_WS2812B_PLCC4_5.0x5.0mm_P3.2mm
- added C17: 100nF, Capacitor_SMD:C_0603_1608Metric, F.Cu at (80.3, 71.2)
- added R5: 10k, Resistor_SMD:R_0402_1005Metric, F.Cu at (83.7, 71.0)
- added R6: 1k, Resistor_SMD:R_0402_1005Metric, F.Cu at (83.7, 73.0)
- added SW1: SW_Push, Tekk_Card_Library:R-667_MIT, F.Cu at (82.2, 67.3)
- moved D11 76.3 mm to (105.4, 115.0)
- moved D12 63.4 mm to (105.7, 96.1)
- moved D10 54.8 mm to (128.5, 115.1)
- moved D8 38.0 mm to (180.6, 114.0)
- moved D9 37.0 mm to (154.4, 114.0)
- moved D6 28.4 mm to (179.9, 77.7)
- moved D7 23.7 mm to (180.7, 95.1)
- moved D5 16.2 mm to (152.5, 76.7)
- moved D4 6.88 mm to (128.1, 75.9)
- moved D3 1.14 mm to (104.9, 76.0)
Connections:
- D10 pad 2: Net-(D10-DOUT) -> unconnected-(D10-DOUT-Pad2)
- D11 pad 2: Net-(D10-DOUT) -> Net-(D11-DIN)
- D11 pad 4: Net-(D10-DOUT) -> Net-(D11-DIN)
- D12 pad 2: Net-(D12-DOUT) -> unconnected-(D12-DOUT-Pad2)
- D12 pad 4: Net-(D10-DOUT) -> Net-(D11-DIN)
