File: electrical/Tekk_Card/flash_boot.kicad_sch (KiCad schematic)
At the start: 5 parts, among them SW1 SW_Push, U5 W25Q64JVSSIQ

Commit message: Continue initial prototype
Parts:
- C17: footprint (none) -> Capacitor_SMD:C_0603_1608Metric
- R5: footprint (none) -> Resistor_SMD:R_0402_1005Metric; Tolerance (none) -> 5%
- R6: footprint (none) -> Resistor_SMD:R_0402_1005Metric
- SW1: footprint (none) -> Tekk_Card_Library:R-667_MIT
Changed lines of the file:
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@@
 			)
 		)
-		(property "Footprint" ""
+		(property "Footprint" "Capacitor_SMD:C_0603_1608Metric"
 			(at 213.0552 72.39 0)
 			(effects
@@
 			)
 		)
-		(property "Footprint" ""
+		(property "Footprint" "Tekk_Card_Library:R-667_MIT"
 			(at 55.88 82.55 0)
 			(effects
@@
 			)
 		)
-		(property "Footprint" ""
+		(property "Footprint" "Resistor_SMD:R_0402_1005Metric"
 			(at 73.914 86.614 90)
 			(effects
@@
 			)
 		)
-		(property "Footprint" ""
+		(property "Footprint" "Resistor_SMD:R_0402_1005Metric"
 			(at 88.646 71.374 90)
 			(effects
@@
 			(at 87.63 71.12 0)
 			(effects
+				(font
+					(size 1.27 1.27)
+				)
+				(hide yes)
+			)
+		)
+		(property "Tolerance" "5%"
+			(at 87.63 71.12 0)
+			(effects
